File: CADandPCB/PCB/armBandShield.sch (EAGLE design)
At the start: 25 parts, among them U1 MPU-9250

Commit message: Rev 1 board completed. Performed checks and added headers for switch.
Parts:
- removed VIN_SWITCH: (no value), SparkFun-Switches:SWITCH-SPDT-SMD-RIGHT-ANGLE
- added SWITCH_HEADERS: 455-1750-1-ND, SparkFun-Connectors:CONN_03
Connections:
- net N$1: now also SWITCH_HEADERS.2; no longer VIN_SWITCH.S
- net VIN: now also SWITCH_HEADERS.1; no longer VIN_SWITCH.P
Changed lines of the file:
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@@
 <part name="P+5" library="supply1" library_urn="urn:adsk.eagle:library:371" deviceset="VCC" device=""/>
 <part name="GND16" library="SparkFun-PowerSymbols" deviceset="GND" device=""/>
-<part name="VIN_SWITCH" library="SparkFun-Switches" deviceset="SWITCH-SPDT" device="-SMD-RIGHT-ANGLE"/>
 <part name="SUPPLY1" library="SparkFun-PowerSymbols" deviceset="VCC_2" device=""/>
 <part name="GND17" library="SparkFun-PowerSymbols" deviceset="GND" device=""/>
@@
 <part name="C3" library="SparkFun-Capacitors" deviceset="0.1UF-25V(+80/-20%)(0603)" device="" value="0.1uF"/>
 <part name="GND22" library="SparkFun-Aesthetics" deviceset="GND" device=""/>
+<part name="SWITCH_HEADERS" library="SparkFun-Connectors" deviceset="CONN_03" device="" value="455-1750-1-ND"/>
 </parts>
 <sheets>
@@
 <attribute name="VALUE" x="137.16" y="-0.254" size="1.778" layer="96" align="top-center"/>
 </instance>
-<instance part="VIN_SWITCH" gate="1" x="180.34" y="0" smashed="yes" rot="R180">
-<attribute name="NAME" x="176.53" y="-5.588" size="1.778" layer="95" font="vector" align="bottom-center"/>
-<attribute name="VALUE" x="179.324" y="3.302" size="1.778" layer="96" font="vector" rot="R180" align="top-center"/>
-</instance>
 <instance part="SUPPLY1" gate="G$1" x="172.72" y="33.02" smashed="yes" rot="R270">
 <attribute name="VALUE" x="178.054" y="30.48" size="1.778" layer="96" align="bottom-center"/>
@@
 <instance part="GND22" gate="1" x="96.52" y="48.26" smashed="yes">
 <attribute name="VALUE" x="93.98" y="45.72" size="1.778" layer="96"/>
+</instance>
+<instance part="SWITCH_HEADERS" gate="J$1" x="180.34" y="-10.16" smashed="yes" rot="R90">
+<attribute name="NAME" x="190.5" y="-13.462" size="1.778" layer="95" font="vector" rot="R180"/>
 </instance>
 </instances>
@@
 </segment>
 <segment>
-<pinref part="VIN_SWITCH" gate="1" pin="P"/>
-<wire x1="182.88" y1="0" x2="185.42" y2="0" width="0.1524" layer="91"/>
-<label x="185.42" y="0" size="1.27" layer="95" xref="yes"/>
+<wire x1="182.88" y1="-2.54" x2="193.04" y2="-2.54" width="0.1524" layer="91"/>
+<label x="193.04" y="-2.54" size="1.27" layer="95" xref="yes"/>
+<pinref part="SWITCH_HEADERS" gate="J$1" pin="1"/>
 </segment>
 </net>
@@
 <net name="N$1" class="0">
 <segment>
-<pinref part="VIN_SWITCH" gate="1" pin="S"/>
 <pinref part="VIN_HEADERS" gate="G$1" pin="1"/>
-<wire x1="175.26" y1="2.54" x2="172.72" y2="2.54" width="0.1524" layer="91"/>
-</segment>
-</net>
+<pinref part="SWITCH_HEADERS" gate="J$1" pin="2"/>
+<wire x1="172.72" y1="2.54" x2="180.34" y2="2.54" width="0.1524" layer="91"/>
+<wire x1="180.34" y1="2.54" x2="180.34" y2="-2.54" width="0.1524" layer="91"/>
+</segment>
+</net>

Commit message: Replace MPU-9250 with MPU-6050. Added logic level. Cleaned up schematic.
Parts:
- removed C1, C2: 0.1uF, SparkFun-Capacitors:0.1UF-25V(+80/-20%)(0603)
- removed MULTIPLEXER_HEADERS: (no value), SparkFun-Connectors:CONN_08"
- removed R11, R12: 10K, SparkFun-Resistors:10KOHM-1/10W-1%(0603)0603
- removed R13: 10k, SparkFun-Resistors:10KOHM-0603-1/10W-1%
- removed U1: MPU-9250, Testing:MPU-9250
- added C4, C7: 0.1uF, SparkFun-Capacitors:0.1UF-25V(+80/-20%)(0603)
- added C5: 10nF, SparkFun-Capacitors:10NF-0603-50V-10%
- added C6: 2.2nF, SparkFun-Capacitors:2.2NF/2200PF-0603-50V-10%
- added FSR_HEADERS: (no value), SparkFun-Connectors:CONN_08"
- added IMU: MPU-6050-1, Testing:MPU-6050-1
- added LLC1, LLC2: BSS138, SparkFun:MOSFET-NCHANNELSMD
- added R16, R17, R20, R21: 10K, SparkFun:RESISTOR0603-RES
- added R18, R19: 10K, SparkFun-Resistors:10KOHM-1/10W-1%(0603)0603
- MULTIPLEXER: value (none) -> 74HC4051
Connections:
- removed net A4/SDA: R11.1, RIGHT_HEADER.8, U1.SDA/SDI
- removed net A5/SCL: R12.1, RIGHT_HEADER.9, U1.SCL/SCLK
- removed net N$2: MULTIPLEXER.!E!, R13.1
- removed net REGOUT: C1.1, U1.REGOUT
- new net A4/SDA/HIGH: LLC1.D, R17.2, RIGHT_HEADER.8
- new net A4/SDA/LOW: IMU.SDA, LLC1.S, R16.2, R18.2
- new net A5/SCL/HIGH: LLC2.D, R21.2, RIGHT_HEADER.9
- new net A5/SCL/LOW: IMU.SCL, LLC2.S, R19.2, R20.2
- new net N$3: C6.1, IMU.CPOUT
- new net N$5: C4.1, IMU.REGOUT
- net FSR1: now also FSR_HEADERS.1; no longer MULTIPLEXER_HEADERS.1
- net FSR2: now also FSR_HEADERS.2; no longer MULTIPLEXER_HEADERS.2
- net FSR3: now also FSR_HEADERS.3; no longer MULTIPLEXER_HEADERS.3
- net FSR4: now also FSR_HEADERS.4; no longer MULTIPLEXER_HEADERS.4
- net FSR5: now also FSR_HEADERS.5; no longer MULTIPLEXER_HEADERS.5
- net FSR6: now also FSR_HEADERS.6; no longer MULTIPLEXER_HEADERS.6
- net FSR7: now also FSR_HEADERS.7; no longer MULTIPLEXER_HEADERS.7
- net FSR8: now also FSR_HEADERS.8; no longer MULTIPLEXER_HEADERS.8
- net GND: now also C4.2, C5.2, C6.2, C7.2, IMU.AD0, IMU.CLKIN, IMU.FSYNC, IMU.GND, MULTIPLEXER.!E!; no longer C1.2, C2.2, R13.2, U1.AD0/SDO, U1.FSYNC, U1.GND
- net VCC: now also R17.1, R21.1
- net VCC_2: now also C5.1, C7.1, IMU.VDD, IMU.VLOGIC, LLC1.G, LLC2.G, R16.1, R18.1, R19.1, R20.1; no longer C2.1, R11.2, R12.2, U1.VDD, U1.VDDIO
Other:
- note added: "1"
- note added: "1. FSR - Force Sensative Resistor - Sparkfun SEN-09673. Attach one end to header and other to VCC. 2. FSR ranges between 1MΩ at low and 2.5kΩ with full pressure. Therefore, voltage divider range varries between 0-3.4 V. 3. VEE set to GND, no bipolar supply. 4. E set to GND to keep enable on."
- note added: "10"
- note added: "2"
- note added: "3"
- note added: "4"
- note added: "5"
- note added: "5. Shield for Arduino Nano V3 footprint. 6. Bluetooth module is HC-05. RX pin on module only supports logic 3.3 V hence the voltage divider. No voltage divider is required for the TX module to RX Arduino connection as high logic is satisfied. 7. VCC header to be used with the FSR's. 8. Two position SPDT switch used as SPST - Sparkfun COM-00102. To be soldered post manufacturing."
- note added: "5.0 V 3.3 V 7-12 V"
- note added: "6"
- note added: "6-DOF Inertial Measurement Unit (IMU) and Logic Level Conversion"
- note added: "7"
- note added: "8"
- note added: "8 Channel Multiplexer and Voltage Dividers for FSR's"
- note added: "9"
- note added: "9. As per MPU-6050 pinout: INT - Interrupt digital output (totem pole or open-drain). Connection is optional. FSYNC - Frame synchronization digital input. Connect to GND if unused. CLKIN - Optional external reference clock input. Connect to GND if unused. AUX_DA - I2C master serial data, for connecting to external sensors. Connection is optional. AUX_CL - I2C Master serial clock, for connecting t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"
- note added: "Pin and Header Assignment"
- note added: "VCC VCC_2 VIN"
- moved on the sheet: BT_HEADERS, C3, LEFT_HEADER, MULTIPLEXER, R1, R10, R2, R3, R4, R5, R6, R7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

Commit message: Added reference designators and double checked entire schematic.
Parts:
- 74HC4051: value 74HC4051 -> U1
- renumbered IMU to U2, LLC1 to Q1, LLC2 to Q2, MULTIPLEXER to 74HC4051
